File: maximiseur3.sch (KiCad schematic (older format))
At the start: 31 parts, among them P1 M- PV- M+ PV+, P2 SW SW, Q1 IRLB3036G, Q2 IRLB3036G, Q3 IRLB3036G, Q4 IRLB3036G, T1 BD139, U1 LM311

Commit message: work in progress
Parts:
- removed P1: M- PV- M+ PV+, maximiseur:bornier4, symbol maximiseur3-rescue:CONN_01X04
- added C10, C7, C8, C9: 1000µF, maximiseur:CP_Radial_D16.0mm_P7.50mm, symbol maximiseur3-rescue:CP2
- added J1: PV+/M+, maximiseur:7808, symbol screw_terminal_01x01:Screw_Terminal_01x01
- added J2: M-, maximiseur:7808, symbol screw_terminal_01x01:Screw_Terminal_01x01
- added J3: PV-, maximiseur:7808, symbol screw_terminal_01x01:Screw_Terminal_01x01
- C3, C4, C5, C6: footprint Capacitor_THT:CP_Radial_D35.0mm_P10.00mm_SnapIn -> maximiseur:CP_Radial_D16.0mm_P7.50mm
- D1, D2, D3, D4: footprint maximiseur:D6.5 -> maximiseur:D_DO-201AE_P15.24mm_Horizontal
- U1: footprint (none) -> maximiseur:DIP-8__300_ELL
- renumbered P2 to P1
Connections:
- wire segments 115 -> 129
Other:
- moved on the sheet: D1, D2, D3, D4, P1, Q1, Q2, Q3, Q4, R10, R7, R8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

Commit message: work in progress
Parts:
- T1: symbol Transistor_BJT:BD139 -> maximiseur3-rescue:BD139-Transistor_BJT
- U1: symbol Comparator:LM311 -> maximiseur3-rescue:LM311-Comparator
Changed lines of the file:
@@
 	1800 1300 4175 1300
 $Comp
-L Transistor_BJT:BD139 T1
+L maximiseur3-rescue:BD139-Transistor_BJT T1
 U 1 1 5D2C4DE3
 P 1350 1650
@@
 	8475 1300 8625 1300
 $Comp
-L Comparator:LM311 U1
+L maximiseur3-rescue:LM311-Comparator U1
 U 1 1 5D4CCDDC
 P 3000 3100

Commit message: work in progress
Parts:
- added C2: 100nF, Capacitor_THT:C_Rect_L7.0mm_W2.0mm_P5.00mm, symbol maximiseur3-rescue:C
- C1: value 0,1µF -> 10µF; footprint Capacitor_THT:C_Disc_D10.0mm_W2.5mm_P5.00mm -> Capacitor_THT:CP_Radial_D5.0mm_P2.50mm
- C3: renamed from C2; footprint maximiseur:C_Rect_L7_W2.5_P5 -> Capacitor_THT:C_Disc_D5.0mm_W2.5mm_P2.50mm
- DZ1, DZ2: footprint maximiseur:D3 -> Diode_THT:D_DO-34_SOD68_P7.62mm_Horizontal
- R1, R10, R2, R4, R5, R6, R7, R8, R9: footprint maximiseur:R3-LARGE_PADS -> Resistor_THT:R_Axial_DIN0207_L6.3mm_D2.5mm_P7.62mm_Horizontal
- R3: value 3k3 -> 2k2; footprint maximiseur:R3-LARGE_PADS -> Resistor_THT:R_Axial_DIN0207_L6.3mm_D2.5mm_P7.62mm_Horizontal
- U1: footprint maximiseur:DIP-8__300_ELL -> Package_DIP:DIP-8_W7.62mm_LongPads
- renumbered C9 to C10, C10 to C11, C3 to C4, C4 to C5, C5 to C6, C6 to C7, C7 to C8, C8 to C9
Connections:
- net PV-: now also C2.2
- net +V renamed +15V
- net +15V: now also C2.1
Changed lines of the file:
@@
 $EndComp
 $Comp
-L maximiseur3-rescue:CP2 C5
+L maximiseur3-rescue:CP2 C6
 U 1 1 55757860
 P 4725 2550
-F 0 "C5" H 4725 2650 40  0000 L CNN
+F 0 "C6" H 4725 2650 40  0000 L CNN
 F 1 "1000µF" H 4731 2465 40  0000 L CNN
 F 2 "maximiseur:CP_Radial_D16.0mm_P7.50mm" H 4763 2400 30  0001 C CNN
@@
 F 0 "R2" V 1880 2450 50  0000 C CNN
 F 1 "15k" V 1800 2450 50  0000 C CNN
-F 2 "maximiseur:R3-LARGE_PADS" V 1730 2450 30  0001 C CNN
+F 2 "Resistor_THT:R_Axial_DIN0207_L6.3mm_D2.5mm_P7.62mm_Horizontal" V 1730 2450 30  0001 C CNN
 F 3 "" H 1800 2450 30  0000 C CNN
 	1    1800 2450
@@
 P 1800 3550
 F 0 "R3" V 1880 3550 50  0000 C CNN
-F 1 "3k3" V 1800 3550 50  0000 C CNN
-F 2 "maximiseur:R3-LARGE_PADS" V 1730 3550 30  0001 C CNN
+F 1 "2k2" V 1800 3550 50  0000 C CNN
+F 2 "Resistor_THT:R_Axial_DIN0207_L6.3mm_D2.5mm_P7.62mm_Horizontal" V 1730 3550 30  0001 C CNN
 F 3 "" H 1800 3550 30  0000 C CNN
 	1    1800 3550
@@
 F 0 "R4" V 2280 2450 50  0000 C CNN
 F 1 "3k3" V 2200 2450 50  0000 C CNN
-F 2 "maximiseur:R3-LARGE_PADS" V 2130 2450 30  0001 C CNN
+F 2 "Resistor_THT:R_Axial_DIN0207_L6.3mm_D2.5mm_P7.62mm_Horizontal" V 2130 2450 30  0001 C CNN
 F 3 "" H 2200 2450 30  0000 C CNN
 	1    2200 2450
@@
 F 0 "R6" V 3780 2150 50  0000 C CNN
 F 1 "1k5" V 3700 2150 50  0000 C CNN
-F 2 "maximiseur:R3-LARGE_PADS" V 3630 2150 30  0001 C CNN
+F 2 "Resistor_THT:R_Axial_DIN0207_L6.3mm_D2.5mm_P7.62mm_Horizontal" V 3630 2150 30  0001 C CNN
 F 3 "" H 3700 2150 30  0000 C CNN
 	1    3700 2150
@@
 F 0 "R5" V 3480 2600 50  0000 C CNN
 F 1 "100k" V 3400 2600 50  0000 C CNN
-F 2 "maximiseur:R3-LARGE_PADS" V 3330 2600 30  0001 C CNN
+F 2 "Resistor_THT:R_Axial_DIN0207_L6.3mm_D2.5mm_P7.62mm_Horizontal" V 3330 2600 30  0001 C CNN
 F 3 "" H 3400 2600 30  0000 C CNN
 	1    3400 2600
@@
 $EndComp
 $Comp
-L maximiseur3-rescue:C C2
+L maximiseur3-rescue:C C3
 U 1 1 55B2142C
 P 3400 2400
-F 0 "C2" V 3350 2450 50  0000 L CNN
+F 0 "C3" V 3350 2450 50  0000 L CNN
 F 1 "100pF" V 3350 2100 50  0000 L CNN
-F 2 "maximiseur:C_Rect_L7_W2.5_P5" H 3438 2250 30  0001 C CNN
+F 2 "Capacitor_THT:C_Disc_D5.0mm_W2.5mm_P2.50mm" H 3438 2250 30  0001 C CNN
 F 3 "" H 3400 2400 60  0000 C CNN
 	1    3400 2400
 	0    1    1    0
-$EndComp
-$Comp
-L maximiseur3-rescue:CP C1
-U 1 1 55B216BE
-P 1450 3550
-F 0 "C1" H 1475 3650 50  0000 L CNN
-F 1 "0,1µF" H 1475 3450 50  0000 L CNN
-F 2 "Capacitor_THT:C_Disc_D10.0mm_W2.5mm_P5.00mm" H 1488 3400 30  0001 C CNN
-F 3 "" H 1450 3550 60  0000 C CNN
-	1    1450 3550
-	1    0    0    -1
 $EndComp
 $Comp
@@
 F 0 "DZ2" H 2200 3700 50  0000 C CNN
 F 1 "6,2V" H 2200 3500 50  0000 C CNN
-F 2 "maximiseur:D3" H 2200 3600 60  0001 C CNN
+F 2 "Diode_THT:D_DO-34_SOD68_P7.62mm_Horizontal" H 2200 3600 60  0001 C CNN
 F 3 "" H 2200 3600 60  0000 C CNN
 	1    2200 3600
@@
 M+
 Text Label 2200 1900 0    60   ~ 0
-+V
++15V
 Wire Wire Line
 	9175 2150 8625 2150
@@
 F 0 "DZ1" H 1079 3679 50  0000 L CNN
 F 1 "15V" H 1025 3500 50  0000 L CNN
-F 2 "maximiseur:D3" H 1125 3600 60  0001 C CNN
+F 2 "Diode_THT:D_DO-34_SOD68_P7.62mm_Horizontal" H 1125 3600 60  0001 C CNN
 F 3 "" H 1125 3600 60  0000 C CNN
 	1    1125 3600
@@
 F 0 "R1" V 1205 1475 50  0000 C CNN
 F 1 "3k3" V 1125 1475 50  0000 C CNN
-F 2 "maximiseur:R3-LARGE_PADS" V 1055 1475 30  0001 C CNN
+F 2 "Resistor_THT:R_Axial_DIN0207_L6.3mm_D2.5mm_P7.62mm_Horizontal" V 1055 1475 30  0001 C CNN
 F 3 "" H 1125 1475 30  0000 C CNN
 	1    1125 1475
@@
 	8475 2450 8000 2450
 $Comp
-L maximiseur3-rescue:CP2 C4
+L maximiseur3-rescue:CP2 C5
 U 1 1 5D2F2FC9
 P 4450 2550
-F 0 "C4" H 4450 2650 40  0000 L CNN
+F 0 "C5" H 4450 2650 40  0000 L CNN
 F 1 "1000µF" H 4456 2465 40  0000 L CNN
 F 2 "maximiseur:CP_Radial_D16.0mm_P7.50mm" H 4488 2400 30  0001 C CNN
@@
 $EndComp
 $Comp
-L maximiseur3-rescue:CP2 C3
+L maximiseur3-rescue:CP2 C4
 U 1 1 5D2F3459
 P 4175 2550
-F 0 "C3" H 4175 2650 40  0000 L CNN
+F 0 "C4" H 4175 2650 40  0000 L CNN
 F 1 "1000µF" H 4181 2465 40  0000 L CNN
 F 2 "maximiseur:CP_Radial_D16.0mm_P7.50mm" H 4213 2400 30  0001 C CNN
@@
 F 0 "R7" V 6780 3300 50  0000 C CNN
 F 1 "150" V 6700 3300 50  0000 C CNN
-F 2 "maximiseur:R3-LARGE_PADS" V 6630 3300 30  0001 C CNN
+F 2 "Resistor_THT:R_Axial_DIN0207_L6.3mm_D2.5mm_P7.62mm_Horizontal" V 6630 3300 30  0001 C CNN
 F 3 "" H 6700 3300 30  0000 C CNN
 	1    6700 3300
@@
 F 0 "R8" V 7255 3300 50  0000 C CNN
 F 1 "150" V 7175 3300 50  0000 C CNN
-F 2 "maximiseur:R3-LARGE_PADS" V 7105 3300 30  0001 C CNN
+F 2 "Resistor_THT:R_Axial_DIN0207_L6.3mm_D2.5mm_P7.62mm_Horizontal" V 7105 3300 30  0001 C CNN
 F 3 "" H 7175 3300 30  0000 C CNN
 	1    7175 3300
@@
 F 0 "R9" V 7780 3300 50  0000 C CNN
 F 1 "150" V 7700 3300 50  0000 C CNN
-F 2 "maximiseur:R3-LARGE_PADS" V 7630 3300 30  0001 C CNN
+F 2 "Resistor_THT:R_Axial_DIN0207_L6.3mm_D2.5mm_P7.62mm_Horizontal" V 7630 3300 30  0001 C CNN
 F 3 "" H 7700 3300 30  0000 C CNN
 	1    7700 3300
@@
 F 0 "R10" V 8255 3300 50  0000 C CNN
 F 1 "150" V 8175 3300 50  0000 C CNN
-F 2 "maximiseur:R3-LARGE_PADS" V 8105 3300 30  0001 C CNN
+F 2 "Resistor_THT:R_Axial_DIN0207_L6.3mm_D2.5mm_P7.62mm_Horizontal" V 8105 3300 30  0001 C CNN
 F 3 "" H 8175 3300 30  0000 C CNN
 	1    8175 3300
@@
 F 0 "U1" H 3344 3146 50  0000 L CNN
 F 1 "LM311" H 3344 3055 50  0000 L CNN
-F 2 "maximiseur:DIP-8__300_ELL" H 3000 3100 50  0001 C CNN
+F 2 "Package_DIP:DIP-8_W7.62mm_LongPads" H 3000 3100 50  0001 C CNN
 F 3 "http://www.ti.com/lit/ds/symlink/lm311.pdf" H 3000 3100 50  0001 C CNN
 	1    3000 3100
@@
 	3300 3100 3700 3100
 Wire Wire Line
-	2900 1900 2900 2800
+	2900 1900 2900 2700
 Wire Wire Line
 	2450 3000 2700 3000
@@
 	2200 3200 2700 3200
 Wire Wire Line
-	2900 3400 2900 4100
+	2900 3400 2900 3700
 Wire Wire Line
 	3000 3400 3000 4100
@@
 	5025 2350 5025 1300
 $Comp
-L maximiseur3-rescue:CP2 C6
+L maximiseur3-rescue:CP2 C7
 U 1 1 557577E2
 P 5025 2550
-F 0 "C6" H 5025 2650 40  0000 L CNN
+F 0 "C7" H 5025 2650 40  0000 L CNN
 F 1 "1000µF" H 5031 2465 40  0000 L CNN
 F 2 "maximiseur:CP_Radial_D16.0mm_P7.50mm" H 5063 2400 30  0001 C CNN
@@
 $EndComp
 $Comp
-L maximiseur3-rescue:CP2 C7
+L maximiseur3-rescue:CP2 C8
 U 1 1 5D5285EA
 P 5300 2550
-F 0 "C7" H 5300 2650 40  0000 L CNN
+F 0 "C8" H 5300 2650 40  0000 L CNN
 F 1 "1000µF" H 5306 2465 40  0000 L CNN
 F 2 "maximiseur:CP_Radial_D16.0mm_P7.50mm" H 5338 2400 30  0001 C CNN
@@
 $EndComp
 $Comp
-L maximiseur3-rescue:CP2 C8
+L maximiseur3-rescue:CP2 C9
 U 1 1 5D5289C3
 P 5575 2550
-F 0 "C8" H 5575 2650 40  0000 L CNN
+F 0 "C9" H 5575 2650 40  0000 L CNN
 F 1 "1000µF" H 5581 2465 40  0000 L CNN
 F 2 "maximiseur:CP_Radial_D16.0mm_P7.50mm" H 5613 2400 30  0001 C CNN
@@
 $EndComp
 $Comp
-L maximiseur3-rescue:CP2 C9
+L maximiseur3-rescue:CP2 C10
 U 1 1 5D528E21
 P 5850 2550
-F 0 "C9" H 5850 2650 40  0000 L CNN
+F 0 "C10" H 5850 2650 40  0000 L CNN
 F 1 "1000µF" H 5856 2465 40  0000 L CNN
 F 2 "maximiseur:CP_Radial_D16.0mm_P7.50mm" H 5888 2400 30  0001 C CNN
@@
 $EndComp
 $Comp
-L maximiseur3-rescue:CP2 C10
+L maximiseur3-rescue:CP2 C11
 U 1 1 5D52925F
 P 6125 2550
-F 0 "C10" H 6125 2650 40  0000 L CNN
+F 0 "C11" H 6125 2650 40  0000 L CNN
 F 1 "1000µF" H 6131 2465 40  0000 L CNN
 F 2 "maximiseur:CP_Radial_D16.0mm_P7.50mm" H 6163 2400 30  0001 C CNN
@@
 Wire Wire Line
 	6125 4100 7000 4100
+$Comp
+L maximiseur3-rescue:CP C1
+U 1 1 55B216BE
+P 1450 3550
+F 0 "C1" H 1475 3650 50  0000 L CNN
+F 1 "10µF" H 1475 3450 50  0000 L CNN
+F 2 "Capacitor_THT:CP_Radial_D5.0mm_P2.50mm" H 1488 3400 30  0001 C CNN
+F 3 "" H 1450 3550 60  0000 C CNN
+	1    1450 3550
+	1    0    0    -1
+$EndComp
+$Comp
+L maximiseur3-rescue:C C2
+U 1 1 5D59BCE0
+P 2650 3450
+F 0 "C2" V 2600 3500 50  0000 L CNN
+F 1 "100nF" V 2600 3150 50  0000 L CNN
+F 2 "Capacitor_THT:C_Rect_L7.0mm_W2.0mm_P5.00mm" H 2688 3300 30  0001 C CNN
+F 3 "" H 2650 3450 60  0000 C CNN
+	1    2650 3450
+	1    0    0    -1
+$EndComp
+Wire Wire Line
+	2650 3300 2650 2700
+Wire Wire Line
+	2650 2700 2900 2700
+Connection ~ 2900 2700
+Wire Wire Line
+	2900 2700 2900 2800
+Wire Wire Line
+	2650 3600 2650 3700
+Wire Wire Line
+	2650 3700 2900 3700
+Connection ~ 2900 3700
+Wire Wire Line
+	2900 3700 2900 4100
 $EndSCHEMATC

Commit message: premiere version correcte du PCB
Parts:
- C3: footprint Capacitor_THT:C_Disc_D5.0mm_W2.5mm_P2.50mm -> Capacitor_THT:C_Rect_L7.0mm_W2.0mm_P5.00mm
- R1, R10, R2, R3, R4, R5, R6, R7, R8, R9: footprint Resistor_THT:R_Axial_DIN0207_L6.3mm_D2.5mm_P7.62mm_Horizontal -> Resistor_THT:R_Axial_DIN0207_L6.3mm_D2.5mm_P10.16mm_Horizontal
Changed lines of the file:
@@
 F 0 "R2" V 1880 2450 50  0000 C CNN
 F 1 "15k" V 1800 2450 50  0000 C CNN
-F 2 "Resistor_THT:R_Axial_DIN0207_L6.3mm_D2.5mm_P7.62mm_Horizontal" V 1730 2450 30  0001 C CNN
+F 2 "Resistor_THT:R_Axial_DIN0207_L6.3mm_D2.5mm_P10.16mm_Horizontal" V 1730 2450 30  0001 C CNN
 F 3 "" H 1800 2450 30  0000 C CNN
 	1    1800 2450
@@
 F 0 "R3" V 1880 3550 50  0000 C CNN
 F 1 "2k2" V 1800 3550 50  0000 C CNN
-F 2 "Resistor_THT:R_Axial_DIN0207_L6.3mm_D2.5mm_P7.62mm_Horizontal" V 1730 3550 30  0001 C CNN
+F 2 "Resistor_THT:R_Axial_DIN0207_L6.3mm_D2.5mm_P10.16mm_Horizontal" V 1730 3550 30  0001 C CNN
 F 3 "" H 1800 3550 30  0000 C CNN
 	1    1800 3550
@@
 F 0 "R4" V 2280 2450 50  0000 C CNN
 F 1 "3k3" V 2200 2450 50  0000 C CNN
-F 2 "Resistor_THT:R_Axial_DIN0207_L6.3mm_D2.5mm_P7.62mm_Horizontal" V 2130 2450 30  0001 C CNN
+F 2 "Resistor_THT:R_Axial_DIN0207_L6.3mm_D2.5mm_P10.16mm_Horizontal" V 2130 2450 30  0001 C CNN
 F 3 "" H 2200 2450 30  0000 C CNN
 	1    2200 2450
@@
 F 0 "R6" V 3780 2150 50  0000 C CNN
 F 1 "1k5" V 3700 2150 50  0000 C CNN
-F 2 "Resistor_THT:R_Axial_DIN0207_L6.3mm_D2.5mm_P7.62mm_Horizontal" V 3630 2150 30  0001 C CNN
+F 2 "Resistor_THT:R_Axial_DIN0207_L6.3mm_D2.5mm_P10.16mm_Horizontal" V 3630 2150 30  0001 C CNN
 F 3 "" H 3700 2150 30  0000 C CNN
 	1    3700 2150
@@
 F 0 "R5" V 3480 2600 50  0000 C CNN
 F 1 "100k" V 3400 2600 50  0000 C CNN
-F 2 "Resistor_THT:R_Axial_DIN0207_L6.3mm_D2.5mm_P7.62mm_Horizontal" V 3330 2600 30  0001 C CNN
+F 2 "Resistor_THT:R_Axial_DIN0207_L6.3mm_D2.5mm_P10.16mm_Horizontal" V 3330 2600 30  0001 C CNN
 F 3 "" H 3400 2600 30  0000 C CNN
 	1    3400 2600
@@
 F 0 "C3" V 3350 2450 50  0000 L CNN
 F 1 "100pF" V 3350 2100 50  0000 L CNN
-F 2 "Capacitor_THT:C_Disc_D5.0mm_W2.5mm_P2.50mm" H 3438 2250 30  0001 C CNN
+F 2 "Capacitor_THT:C_Rect_L7.0mm_W2.0mm_P5.00mm" H 3438 2250 30  0001 C CNN
 F 3 "" H 3400 2400 60  0000 C CNN
 	1    3400 2400
@@
 F 0 "R1" V 1205 1475 50  0000 C CNN
 F 1 "3k3" V 1125 1475 50  0000 C CNN
-F 2 "Resistor_THT:R_Axial_DIN0207_L6.3mm_D2.5mm_P7.62mm_Horizontal" V 1055 1475 30  0001 C CNN
+F 2 "Resistor_THT:R_Axial_DIN0207_L6.3mm_D2.5mm_P10.16mm_Horizontal" V 1055 1475 30  0001 C CNN
 F 3 "" H 1125 1475 30  0000 C CNN
 	1    1125 1475
@@
 F 0 "R7" V 6780 3300 50  0000 C CNN
 F 1 "150" V 6700 3300 50  0000 C CNN
-F 2 "Resistor_THT:R_Axial_DIN0207_L6.3mm_D2.5mm_P7.62mm_Horizontal" V 6630 3300 30  0001 C CNN
+F 2 "Resistor_THT:R_Axial_DIN0207_L6.3mm_D2.5mm_P10.16mm_Horizontal" V 6630 3300 30  0001 C CNN
 F 3 "" H 6700 3300 30  0000 C CNN
 	1    6700 3300
@@
 F 0 "R8" V 7255 3300 50  0000 C CNN
 F 1 "150" V 7175 3300 50  0000 C CNN
-F 2 "Resistor_THT:R_Axial_DIN0207_L6.3mm_D2.5mm_P7.62mm_Horizontal" V 7105 3300 30  0001 C CNN
+F 2 "Resistor_THT:R_Axial_DIN0207_L6.3mm_D2.5mm_P10.16mm_Horizontal" V 7105 3300 30  0001 C CNN
 F 3 "" H 7175 3300 30  0000 C CNN
 	1    7175 3300
@@
 F 0 "R9" V 7780 3300 50  0000 C CNN
 F 1 "150" V 7700 3300 50  0000 C CNN
-F 2 "Resistor_THT:R_Axial_DIN0207_L6.3mm_D2.5mm_P7.62mm_Horizontal" V 7630 3300 30  0001 C CNN
+F 2 "Resistor_THT:R_Axial_DIN0207_L6.3mm_D2.5mm_P10.16mm_Horizontal" V 7630 3300 30  0001 C CNN
 F 3 "" H 7700 3300 30  0000 C CNN
 	1    7700 3300
@@
 F 0 "R10" V 8255 3300 50  0000 C CNN
 F 1 "150" V 8175 3300 50  0000 C CNN
-F 2 "Resistor_THT:R_Axial_DIN0207_L6.3mm_D2.5mm_P7.62mm_Horizontal" V 8105 3300 30  0001 C CNN
+F 2 "Resistor_THT:R_Axial_DIN0207_L6.3mm_D2.5mm_P10.16mm_Horizontal" V 8105 3300 30  0001 C CNN
 F 3 "" H 8175 3300 30  0000 C CNN
 	1    8175 3300
